Commit message: the urdf is ready for champ, but cant run setup assistant since it is for ros1, will import the setup files as is and add custom ros2 controll using a git repo i found

File: install/champbot_nodes/share/champbot_nodes/urdf/robot.urdf.xacro (robot description, xacro)
@@ -188,35 +188,9 @@
   <xacro:leg prefix="lh" px="${-hip_x}" py="${ hip_y}" ydir="1"/>
   <xacro:leg prefix="rh" px="${-hip_x}" py="${-hip_y}" ydir="-1"/>
-  <!-- ============================ ros2_control ========================= -->
-  <!-- POSITION command interface (stands rigidly for viewing). When CHAMP is
-       wired up it brings its own controllers - this is just so the bare robot
-       can be spawned and stood up on its own. -->
-  <xacro:macro name="leg_ctrl" params="prefix">
-    <joint name="${prefix}_hip_joint">
-      <command_interface name="position"/>
-      <state_interface name="position"><param name="initial_value">0.0</param></state_interface>
-    </joint>
-    <joint name="${prefix}_upper_leg_joint">
-      <command_interface name="position"/>
-      <state_interface name="position"><param name="initial_value">0.0</param></state_interface>
-    </joint>
-    <joint name="${prefix}_lower_leg_joint">
-      <command_interface name="position"/>
-      <state_interface name="position"><param name="initial_value">0.0</param></state_interface>
-    </joint>
-  </xacro:macro>
-  <ros2_control name="GazeboSystem" type="system">
-    <hardware>
-      <plugin>gazebo_ros2_control/GazeboSystem</plugin>
-    </hardware>
-    <xacro:leg_ctrl prefix="lf"/>
-    <xacro:leg_ctrl prefix="rf"/>
-    <xacro:leg_ctrl prefix="lh"/>
-    <xacro:leg_ctrl prefix="rh"/>
-  </ros2_control>
-  <gazebo>
-    <plugin filename="libgazebo_ros2_control.so" name="gazebo_ros2_control">
-      <parameters>$(find quadbot_nodes)/config/quadbot_controllers.yaml</parameters>
-    </plugin>
-  </gazebo>
+  <!-- NOTE: No ros2_control / gazebo_ros2_control block here on purpose.
+       The CHAMP setup assistant only needs the kinematic chain (links + joints)
+       from robot_description, and CHAMP generates its own controllers and
+       gazebo bringup later. The old gazebo_ros2_control plugin (which pointed
+       at $(find quadbot_nodes)/config/...) was removed because that package
+       does not exist in this workspace and it broke xacro expansion. -->
 </robot>

Commit message: feet are now spheres and carry no mass so closer to the original and better design, still stable

File: install/champbot_nodes/share/champbot_nodes/urdf/robot.urdf.xacro (robot description, xacro)
@@ -162,17 +162,12 @@
     <link name="${prefix}_foot_link">
       <visual>
-        <origin xyz="0 0 -0.0175" rpy="0 0 0"/>
-        <geometry><box size="0.045 0.05 0.035"/></geometry>
+        <origin xyz="0 0 0" rpy="0 0 0"/>
+        <geometry><sphere radius="${foot_rad}"/></geometry>
         <material name="foot_grey"/>
       </visual>
       <collision>
-        <origin xyz="0 0 -0.0175" rpy="0 0 0"/>
-        <geometry><box size="0.045 0.05 0.035"/></geometry>
-      </collision>
-      <inertial>
-        <origin xyz="0 0 -0.0175" rpy="0 0 0"/>
-        <mass value="0.05"/>
-        <xacro:box_inertia m="0.05" x="0.045" y="0.05" z="0.035"/>
-      </inertial>
+        <origin xyz="0 0 0" rpy="0 0 0"/>
+        <geometry><sphere radius="${foot_rad}"/></geometry>
+      </collision>
     </link>
     <gazebo reference="${prefix}_foot_link">

Commit message: bigger hip x and y to be more stable

File: install/champbot_nodes/share/champbot_nodes/urdf/robot.urdf.xacro (robot description, xacro)
@@ -20,6 +20,6 @@
   <xacro:property name="leg_rad"   value="0.018"/>
   <xacro:property name="foot_rad"  value="0.025"/>
-  <xacro:property name="hip_x" value="0.14"/>
-  <xacro:property name="hip_y" value="0.09"/>
+  <xacro:property name="hip_x" value="0.175"/>
+  <xacro:property name="hip_y" value="0.105"/>
   <xacro:property name="hip_z" value="-0.02"/>
   <xacro:property name="j_eff" value="40.0"/>
@@ -176,5 +176,5 @@
       <kp>100000.0</kp>
       <kd>2.0</kd>
-      <minDepth>0.002</minDepth>
+      <minDepth>0.001</minDepth>
     </gazebo>
   </xacro:macro>

Commit message: wider body, better stabillity

File: install/champbot_nodes/share/champbot_nodes/urdf/robot.urdf.xacro (robot description, xacro)
@@ -12,5 +12,5 @@
   <!-- ============================ dimensions ============================ -->
   <xacro:property name="body_len"  value="0.40"/>
-  <xacro:property name="body_wid"  value="0.18"/>
+  <xacro:property name="body_wid"  value="0.26"/>
   <xacro:property name="body_hgt"  value="0.08"/>
   <xacro:property name="body_mass" value="3.0"/>
@@ -19,5 +19,5 @@
   <xacro:property name="lower_len" value="0.14"/>
   <xacro:property name="leg_rad"   value="0.018"/>
-  <xacro:property name="foot_rad"  value="0.025"/>
+  <xacro:property name="foot_rad"  value="0.018"/>
   <xacro:property name="hip_x" value="0.175"/>
   <xacro:property name="hip_y" value="0.105"/>

Commit message: nominal height higher, moves alot better no lag like before

File: install/champbot_nodes/share/champbot_nodes/urdf/robot.urdf.xacro (robot description, xacro)
@@ -11,5 +11,5 @@
 <robot name="quadbot" xmlns:xacro="http://www.ros.org/wiki/xacro">
   <!-- ============================ dimensions ============================ -->
-  <xacro:property name="body_len"  value="0.40"/>
+  <xacro:property name="body_len"  value="0.50"/>
   <xacro:property name="body_wid"  value="0.26"/>
   <xacro:property name="body_hgt"  value="0.08"/>

Commit message: best all around version for movement, still some slight modifications are needed before Lidar

File: install/champbot_nodes/share/champbot_nodes/urdf/robot.urdf.xacro (robot description, xacro)
@@ -19,5 +19,5 @@
   <xacro:property name="lower_len" value="0.14"/>
   <xacro:property name="leg_rad"   value="0.018"/>
-  <xacro:property name="foot_rad"  value="0.018"/>
+  <xacro:property name="foot_rad"  value="0.013"/>
   <xacro:property name="hip_x" value="0.175"/>
   <xacro:property name="hip_y" value="0.105"/>

Commit message: ver smooth movement , the j_eff and j_vel limits were the main culprits, they were reduced

File: install/champbot_nodes/share/champbot_nodes/urdf/robot.urdf.xacro (robot description, xacro)
@@ -23,6 +23,6 @@
   <xacro:property name="hip_y" value="0.105"/>
   <xacro:property name="hip_z" value="-0.02"/>
-  <xacro:property name="j_eff" value="40.0"/>
-  <xacro:property name="j_vel" value="12.0"/>
+  <xacro:property name="j_eff" value="25.0"/>
+  <xacro:property name="j_vel" value="1.5"/>
   <!-- ============================ materials ============================= -->
   <material name="body_blue"><color rgba="0.15 0.35 0.85 1"/></material>
@@ -174,6 +174,6 @@
       <mu1>1.2</mu1>
       <mu2>1.2</mu2>
-      <kp>100000.0</kp>
-      <kd>2.0</kd>
+      <kp>10000.0</kp>
+      <kd>3.0</kd>
       <minDepth>0.001</minDepth>
     </gazebo>

Commit message: added world and rviz tabs

File: install/champbot_nodes/share/champbot_nodes/urdf/robot.urdf.xacro (robot description, xacro)
@@ -183,4 +183,49 @@
   <xacro:leg prefix="lh" px="${-hip_x}" py="${ hip_y}" ydir="1"/>
   <xacro:leg prefix="rh" px="${-hip_x}" py="${-hip_y}" ydir="-1"/>
+  <!-- LIDAR  -->
+  <link name="lidar_link">
+    <visual>
+      <origin xyz="0 0 0" rpy="0 0 0"/>
+      <geometry><cylinder radius="0.06" length="0.03"/></geometry>
+      <material name="joint_yellow"/>
+    </visual>
+    <inertial>
+      <mass value="0.1"/>
+      <xacro:cyl_inertia m="0.1" r="0.03" l="0.02"/>
+    </inertial>
+  </link>
+  <joint name="lidar_joint" type="fixed">
+    <parent link="base_link"/>
+    <child  link="lidar_link"/>
+    <origin xyz="0 0 0.05" rpy="0 0 0"/>
+  </joint>
+  <gazebo reference="lidar_link">
+        <sensor type="ray" name="lidar">
+            <pose>0 0 0 0 0 0</pose>
+            <always_on>true</always_on>
+            <visualize>true</visualize>
+            <update_rate>10</update_rate>
+            <ray>
+            <scan>
+                <horizontal>
+                <samples>360</samples>
+                <min_angle>-3.14159</min_angle>
+                <max_angle>3.14159</max_angle>
+                </horizontal>
+            </scan>
+            <range>
+                <min>0.15</min>
+                <max>12.0</max>
+            </range>
+            </ray>
+            <plugin name="lidar_plugin" filename="libgazebo_ros_ray_sensor.so">
+            <ros>
+                <remapping>~/out:=scan</remapping>
+            </ros>
+            <output_type>sensor_msgs/LaserScan</output_type>
+            <frame_name>lidar_link</frame_name>
+            </plugin>
+        </sensor>
+    </gazebo>
   <!-- ===================================================================== -->
   <!-- CHAMP / Gazebo integration (mirrors chvmp go2_description/xacro).      -->
